File: smartkey-dc-pwm-60w.sch (KiCad schematic (older format))
At the start: 27 parts, among them J3 IN_OUT, J4 Conn_01x06_Female, K1 SANYOU_SRD_Form_C, Q1 SS8050-G, Q2 NCE4009S, SW1 SW_Push, U1 ESP-07S, U2 CJ7805, U3 AMS1117-3.3

Commit message: 新增正确pdf及原理图
Parts:
- added Q?: NCE6080K, Package_TO_SOT_SMD:TO-252-2, symbol Device:Q_NMOS_GDS
- added R? (x2): 10k, Resistor_SMD:R_0603_1608Metric, symbol Device:R
Connections:
- net GND: now also Q?.3 (S), R?.2
- net LED-: now also Q?.2 (D)
- net PWM: now also R?.2
- new net: Q?.1 (G), R?.1, R?.1
Other:
- moved on the sheet: Q2, R7, R8
Changed lines of the file:
@@
 L Device:Q_NMOS_GSD Q2
 U 1 1 627EA7DB
-P 9180 5470
-F 0 "Q2" H 9384 5516 50  0000 L CNN
-F 1 "NCE4009S" H 9384 5425 50  0000 L CNN
-F 2 "Package_TO_SOT_SMD:TO-252-2" H 9380 5570 50  0001 C CNN
-F 3 "~" H 9180 5470 50  0001 C CNN
-	1    9180 5470
+P 8670 5340
+F 0 "Q2" H 8874 5386 50  0000 L CNN
+F 1 "NCE4009S" H 8874 5295 50  0000 L CNN
+F 2 "Package_TO_SOT_SMD:TO-252-2" H 8870 5440 50  0001 C CNN
+F 3 "~" H 8670 5340 50  0001 C CNN
+	1    8670 5340
 	1    0    0    -1
 $EndComp
@@
 L Device:R R8
 U 1 1 627EC39F
-P 8980 5620
-F 0 "R8" H 9050 5666 50  0000 L CNN
-F 1 "10k" H 9050 5575 50  0000 L CNN
-F 2 "Resistor_SMD:R_0603_1608Metric" V 8910 5620 50  0001 C CNN
-F 3 "~" H 8980 5620 50  0001 C CNN
-	1    8980 5620
-	1    0    0    -1
-$EndComp
-Wire Wire Line
-	9280 5670 9280 5770
-Wire Wire Line
-	9280 5770 8980 5770
-Wire Wire Line
-	8980 5470 8850 5470
-Connection ~ 8980 5470
+P 8470 5490
+F 0 "R8" H 8540 5536 50  0000 L CNN
+F 1 "10k" H 8540 5445 50  0000 L CNN
+F 2 "Resistor_SMD:R_0603_1608Metric" V 8400 5490 50  0001 C CNN
+F 3 "~" H 8470 5490 50  0001 C CNN
+	1    8470 5490
+	1    0    0    -1
+$EndComp
+Wire Wire Line
+	8770 5540 8770 5640
+Wire Wire Line
+	8770 5640 8470 5640
+Wire Wire Line
+	8470 5340 8340 5340
+Connection ~ 8470 5340
 $Comp
 L Device:R R7
 U 1 1 627EEFEB
-P 8700 5470
-F 0 "R7" V 8493 5470 50  0000 C CNN
-F 1 "10k" V 8584 5470 50  0000 C CNN
-F 2 "Resistor_SMD:R_0603_1608Metric" V 8630 5470 50  0001 C CNN
-F 3 "~" H 8700 5470 50  0001 C CNN
-	1    8700 5470
+P 8190 5340
+F 0 "R7" V 7983 5340 50  0000 C CNN
+F 1 "10k" V 8074 5340 50  0000 C CNN
+F 2 "Resistor_SMD:R_0603_1608Metric" V 8120 5340 50  0001 C CNN
+F 3 "~" H 8190 5340 50  0001 C CNN
+	1    8190 5340
 	0    1    1    0
 $EndComp
-Text GLabel 8550 5470 0    50   Input ~ 0
+Text GLabel 8040 5340 0    50   Input ~ 0
 PWM
 Wire Wire Line
-	9280 5270 9280 5140
+	8770 5140 8770 5010
 Text GLabel 6430 5620 0    50   Input ~ 0
 VCC+
@@
 Text GLabel 1110 5120 3    50   Input ~ 0
 LED+
-Text GLabel 9280 5140 1    50   Input ~ 0
+Text GLabel 8770 5010 1    50   Input ~ 0
 LED-
 $Comp
 L power:GND #PWR0118
 U 1 1 6286EFEA
-P 9280 5770
-F 0 "#PWR0118" H 9280 5520 50  0001 C CNN
-F 1 "GND" H 9285 5597 50  0000 C CNN
-F 2 "" H 9280 5770 50  0001 C CNN
-F 3 "" H 9280 5770 50  0001 C CNN
-	1    9280 5770
-	1    0    0    -1
-$EndComp
-Connection ~ 9280 5770
+P 8770 5640
+F 0 "#PWR0118" H 8770 5390 50  0001 C CNN
+F 1 "GND" H 8775 5467 50  0000 C CNN
+F 2 "" H 8770 5640 50  0001 C CNN
+F 3 "" H 8770 5640 50  0001 C CNN
+	1    8770 5640
+	1    0    0    -1
+$EndComp
+Connection ~ 8770 5640
 Wire Wire Line
 	2170 1690 2170 1540
@@
 Wire Notes Line
 	490  490  11180 490
+$Comp
+L Device:Q_NMOS_GDS Q?
+U 1 1 62B3ED09
+P 10310 5280
+F 0 "Q?" H 10514 5326 50  0000 L CNN
+F 1 "NCE6080K" H 10514 5235 50  0000 L CNN
+F 2 "Package_TO_SOT_SMD:TO-252-2" H 10510 5380 50  0001 C CNN
+F 3 "~" H 10310 5280 50  0001 C CNN
+	1    10310 5280
+	1    0    0    -1
+$EndComp
+$Comp
+L Device:R R?
+U 1 1 62B44AF3
+P 10110 5430
+F 0 "R?" H 10180 5476 50  0000 L CNN
+F 1 "10k" H 10180 5385 50  0000 L CNN
+F 2 "Resistor_SMD:R_0603_1608Metric" V 10040 5430 50  0001 C CNN
+F 3 "~" H 10110 5430 50  0001 C CNN
+	1    10110 5430
+	1    0    0    -1
+$EndComp
+Wire Wire Line
+	10410 5480 10410 5580
+Wire Wire Line
+	10410 5580 10110 5580
+Wire Wire Line
+	10110 5280 9980 5280
+Connection ~ 10110 5280
+$Comp
+L Device:R R?
+U 1 1 62B44AFD
+P 9830 5280
+F 0 "R?" V 9623 5280 50  0000 C CNN
+F 1 "10k" V 9714 5280 50  0000 C CNN
+F 2 "Resistor_SMD:R_0603_1608Metric" V 9760 5280 50  0001 C CNN
+F 3 "~" H 9830 5280 50  0001 C CNN
+	1    9830 5280
+	0    1    1    0
+$EndComp
+Text GLabel 9680 5280 0    50   Input ~ 0
+PWM
+Wire Wire Line
+	10410 5080 10410 4950
+Text GLabel 10410 4950 1    50   Input ~ 0
+LED-
+$Comp
+L power:GND #PWR?
+U 1 1 62B44B06
+P 10410 5580
+F 0 "#PWR?" H 10410 5330 50  0001 C CNN
+F 1 "GND" H 10415 5407 50  0000 C CNN
+F 2 "" H 10410 5580 50  0001 C CNN
+F 3 "" H 10410 5580 50  0001 C CNN
+	1    10410 5580
+	1    0    0    -1
+$EndComp
+Connection ~ 10410 5580
 $EndSCHEMATC
